Commit message: modify

File: model/robot.xacro (robot description, xacro)
@@ -1,6 +1,4 @@
 <?xml version="1.0"?>
 <robot name="rw" xmlns:xacro="http://www.ros.org/wiki/xacro">
-    <xacro:include filename="$(find xarm_description)/urdf/xarm6/xarm6_robot_macro.xacro" />
-    <xacro:xarm6_urdf prefix="xarm_" />
     <!-- Robot Parameters -->
     <xacro:property name="PI" value="3.14159265"/>
@@ -81,12 +79,4 @@
         <mu2>1.0</mu2>
     </gazebo>
-    <!-- Instantiate xArm6 -->
-    <xacro:xarm6_urdf prefix="xarm_" />
-    <!-- Joint to attach xArm6 to base_link -->
-    <joint name="base_to_xarm_joint" type="fixed">
-        <origin xyz="0.48 0 0.5" rpy="0 0 0" />
-        <parent link="base_link" />
-        <child link="xarm_link_base" />
-    </joint>
     <!-- BASE_FOOTPRINT LINK -->
     <!-- <joint name="base_footprint_joint" type="fixed">

Commit message: add

File: model/robot.xacro (robot description, xacro)
@@ -1,4 +1,6 @@
 <?xml version="1.0"?>
 <robot name="rw" xmlns:xacro="http://www.ros.org/wiki/xacro">
+    <xacro:include filename="$(find xarm_description)/urdf/xarm6/xarm6_robot_macro.xacro" />
+    <xacro:xarm6_urdf prefix="xarm_" />
     <!-- Robot Parameters -->
     <xacro:property name="PI" value="3.14159265"/>
@@ -79,4 +81,12 @@
         <mu2>1.0</mu2>
     </gazebo>
+    <!-- Instantiate xArm6 -->
+    <xacro:xarm6_urdf prefix="xarm_" />
+    <!-- Joint to attach xArm6 to base_link -->
+    <joint name="base_to_xarm_joint" type="fixed">
+        <origin xyz="0.48 0 0.5" rpy="0 0 0" />
+        <parent link="base_link" />
+        <child link="xarm_link_base" />
+    </joint>
     <!-- BASE_FOOTPRINT LINK -->
     <!-- <joint name="base_footprint_joint" type="fixed">

File: srdf/rw_macro.srdf.xacro (robot description, xacro)
@@ -3,5 +3,5 @@
   This is a format for representing semantic information about the robot structure.
   A URDF file must exist for this robot as well, where the joints and the links that are referenced are defined -->
-<robot xmlns:xacro="http://ros.org/wiki/xacro" name="mbot_srdf">
+<robot xmlns:xacro="http://ros.org/wiki/xacro" name="rw_srdf">
   <!-- GROUPS: Representation of a set of joints and links. This can be useful for specifying DOF to plan for, defining arms, end effectors, etc -->
   <!-- LINKS: When a link is specified, the parent joint of that link (if it exists) is automatically included -->
@@ -9,14 +9,14 @@
   <!-- CHAINS: When a chain is specified, all the links along the chain (including endpoints) are included in the group. Additionally, all the joints that are parents to included links are also included. This means that joints along the chain and the parent joint of the base link are included in the group -->
   <!-- SUBGROUPS: Groups can also be formed by referencing to already defined group names -->
-  <xacro:macro name="mbot_macro_srdf" params="prefix=''">
-    <!-- <group name="mbot">
+  <xacro:macro name="rw_macro_srdf" params="prefix=''">
+    <!-- <group name="rw">
       <joint name="left_wheel_joint" />
       <joint name="right_wheel_joint" />
     </group>
-    <group_state name="home" group="mbot">
+    <group_state name="home" group="rw">
       <joint name="left_wheel_joint" value="0" />
       <joint name="right_wheel_joint" value="0" />
     </group_state>
-    <group_state name="test" group="mbot">
+    <group_state name="test" group="rw">
       <joint name="left_wheel_joint" value="1.0" />
       <joint name="right_wheel_joint" value="1.0" />

File: urdf/rw.gazebo.xacro (robot description, xacro)
@@ -1,5 +1,5 @@
 <?xml version="1.0"?>
-<robot name="mbot" xmlns:xacro="http://www.ros.org/wiki/xacro">
-  <xacro:macro name="mbot_gazebo" params="">
+<robot name="rw" xmlns:xacro="http://www.ros.org/wiki/xacro">
+  <xacro:macro name="rw_gazebo" params="">
     <gazebo reference="base_footprint">
       <turnGravityOff>false</turnGravityOff>

File: urdf/rw.ros2_control.xacro (robot description, xacro)
@@ -1,6 +1,6 @@
 <?xml version="1.0"?>
-<robot name="mbot" xmlns:xacro="http://www.ros.org/wiki/xacro">
-  <xacro:macro name="mbot_ros2_control" params="ros2_control_plugin:='uf_robot_hardware/UFRobotFakeSystemHardware'">
-    <ros2_control name="mbot_ros2_control" type="system">
+<robot name="rw" xmlns:xacro="http://www.ros.org/wiki/xacro">
+  <xacro:macro name="rw_ros2_control" params="ros2_control_plugin:='uf_robot_hardware/UFRobotFakeSystemHardware'">
+    <ros2_control name="rw_ros2_control" type="system">
       <hardware>
         <plugin>${ros2_control_plugin}</plugin>

File: urdf/rw.transmission.xacro (robot description, xacro)
@@ -1,6 +1,6 @@
 <?xml version="1.0"?>
-<robot name="mbot" xmlns:xacro="http://www.ros.org/wiki/xacro">
-  <xacro:macro name="mbot_transmission" params="hard_interface:='PositionJointInterface'">
-  <!-- <xacro:macro name="mbot_transmission" params="hard_interface:='VelocityJointInterface'"> -->
+<robot name="rw" xmlns:xacro="http://www.ros.org/wiki/xacro">
+  <xacro:macro name="rw_transmission" params="hard_interface:='PositionJointInterface'">
+  <!-- <xacro:macro name="rw_transmission" params="hard_interface:='VelocityJointInterface'"> -->
     <!-- Transmission is important to link the joints and the controller -->
     <transmission name="left_wheel_joint_trans">

File: urdf/rw.urdf.xacro (robot description, xacro)
@@ -1,4 +1,4 @@
 <?xml version="1.0"?>
-<robot name="mbot" xmlns:xacro="http://www.ros.org/wiki/xacro">
+<robot name="rw" xmlns:xacro="http://www.ros.org/wiki/xacro">
   <!-- PROPERTY LIST -->
   <xacro:property name="M_PI" value="3.1415926"/>
@@ -92,5 +92,5 @@
     </link>
   </xacro:macro>
-  <xacro:macro name="mbot_urdf">
+  <xacro:macro name="rw_urdf">
     <link name="base_footprint">
       <visual>

File: urdf/rw_macro.xacro (robot description, xacro)
@@ -1,19 +1,19 @@
 <?xml version="1.0"?>
-<robot name="mbot" xmlns:xacro="http://www.ros.org/wiki/xacro">
-  <xacro:macro name="mbot_macro" params="ros2_control_plugin:='uf_robot_hardware/UFRobotSystemHardware'">
-    <xacro:include filename="$(find mbot_demo)/urdf/mbot.urdf.xacro" />
-    <xacro:mbot_urdf/>
-    <xacro:include filename="$(find mbot_demo)/urdf/mbot.transmission.xacro" />
-    <xacro:mbot_transmission hard_interface="VelocityJointInterface" />
-    <xacro:include filename="$(find mbot_demo)/urdf/mbot.ros2_control.xacro" />
+<robot name="rw" xmlns:xacro="http://www.ros.org/wiki/xacro">
+  <xacro:macro name="rw_macro" params="ros2_control_plugin:='uf_robot_hardware/UFRobotSystemHardware'">
+    <xacro:include filename="$(find rw)/urdf/rw.urdf.xacro" />
+    <xacro:rw_urdf/>
+    <xacro:include filename="$(find rw)/urdf/rw.transmission.xacro" />
+    <xacro:rw_transmission hard_interface="VelocityJointInterface" />
+    <xacro:include filename="$(find rw)/urdf/rw.ros2_control.xacro" />
     <xacro:if value="${ros2_control_plugin == 'uf_robot_hardware/UFRobotSystemHardware'}">
       <!-- uf_robot_hardware/UFRobotSystemHardware only use on the real xarm robot -->
-      <xacro:mbot_ros2_control ros2_control_plugin="uf_robot_hardware/UFRobotFakeSystemHardware" />
+      <xacro:rw_ros2_control ros2_control_plugin="uf_robot_hardware/UFRobotFakeSystemHardware" />
     </xacro:if>
     <xacro:unless value="${ros2_control_plugin == 'uf_robot_hardware/UFRobotSystemHardware'}">
-      <xacro:mbot_ros2_control ros2_control_plugin="${ros2_control_plugin}" />
+      <xacro:rw_ros2_control ros2_control_plugin="${ros2_control_plugin}" />
     </xacro:unless>
-    <xacro:include filename="$(find mbot_demo)/urdf/mbot.gazebo.xacro" />
-    <xacro:mbot_gazebo/>
+    <xacro:include filename="$(find rw)/urdf/rw.gazebo.xacro" />
+    <xacro:rw_gazebo/>
   </xacro:macro>
 </robot>

File: urdf/rw_with_xarm.urdf.xacro (robot description, xacro)
@@ -1,4 +1,4 @@
 <?xml version="1.0"?>
-<robot name="mbot_with_xarm" xmlns:xacro="http://www.ros.org/wiki/xacro">
+<robot name="rw_with_xarm" xmlns:xacro="http://www.ros.org/wiki/xacro">
   <xacro:arg name="prefix" default=""/>
   <xacro:arg name="hw_ns" default="xarm"/>
@@ -39,6 +39,6 @@
   <xacro:arg name="mesh_suffix" default="stl"/>
   <xacro:arg name="kinematics_suffix" default=""/>
-  <xacro:include filename="$(find mbot_demo)/urdf/mbot_macro.xacro" />
-  <xacro:mbot_macro ros2_control_plugin="$(arg ros2_control_plugin)" />
+  <xacro:include filename="$(find rw)/urdf/rw_macro.xacro" />
+  <xacro:rw_macro ros2_control_plugin="$(arg ros2_control_plugin)" />
   <!-- load xarm device -->
   <xacro:include filename="$(find xarm_description)/urdf/xarm_device_macro.xacro" />
